File: wiring/ardipool/ardipool.kicad_pcb (KiCad board)
At the start: 2 copper layers, 205.7 x 137.2 mm, 23 parts, among them K1 filter, K2 ph, P1 Digital, P10 CONN_01X01, P11 CONN_01X01, P12 CONN_01X01, P13 CONN_01X01, P2 Power, P3 Analog, P4 Analog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

Commit message: update
Parts:
- removed DS1: WC1602A, Display:WC1602A
- removed K1: filter, Relay_THT:Relay_SPDT_SANYOU_SRD_Series_Form_C
- removed K2: ph, Relay_THT:Relay_SPDT_SANYOU_SRD_Series_Form_C
- removed P5: PWM, Socket_Arduino_Mega:Socket_Strip_Arduino_1x10
- removed SW1: SW_Push_Dual, Button_Switch_THT:SW_PUSH_6mm_H5mm
- added Q1: BC557, Package_TO_SOT_THT:TO-92_Inline_Wide, F.Cu at (136.5, 96.5)
- added U5: TXS0108EPW, Package_SO:TSSOP-20_4.4x6.5mm_P0.65mm, F.Cu at (120.0, 97.3)
- added U6: ADS1115IDGS, Package_SO:TSSOP-10_3x3mm_P0.5mm, F.Cu at (127.8, 95.6)
- R2: value 220 -> 1K
- U3: value DHT11 -> ESP32devkitC; footprint Sensor:Aosong_DHT11_5.5x12.0_P2.54mm -> Package_DIP:DIP-40_W25.4mm_Socket_LongPads
- U4: value DS1307+ -> DS3231M; footprint Package_DIP:DIP-8_W7.62mm -> Package_SO:SOIC-16W_7.5x10.3mm_P1.27mm
- moved U3 165.0 mm to (91.9, 77.2), turned to 180 degrees
- moved U4 163.1 mm to (90.0, 99.2)
Connections:
- R1 pad 2: +5V -> +3V3
- R2 pad 1: LCDLED -> Net-(Q1-Pad2)
- R2 pad 2: Net-(DS1-Pad15) -> LED_32
- U1 pad 3: +5V -> +3V3
- U2 pad 3: +5V -> +3V3
- U3 pad 1: +5V -> Net-(U3-Pad1)
- U3 pad 2: DHT -> Net-(U3-Pad2)
- U3 pad 4: GND -> LED_32
- U4 pad 2: Net-(U4-Pad2) -> +3V3
- U4 pad 4: GND -> Net-(U4-Pad4)
- U4 pad 5: SCL -> GND
- U4 pad 6: SDA -> GND
- U4 pad 7: Net-(U4-Pad7) -> GND
- U4 pad 8: +5V -> GND
Routing:
- net Net-(DS1-Pad15): track 81.9 -> 0.00 mm
- net LED_32: track 0.00 -> 81.9 mm
- net SDA: track 0.00 -> 69.0 mm
